File: athene-pcb.kicad_pcb (KiCad board)
At the start: 2 copper layers, 303.2 x 92.1 mm, 162 parts, among them J1 HRO-TYPE-C-31-M-12, K1 KEYSW, K10 KEYSW, K11 KEYSW, K12 KEYSW, K13 KEYSW, K14 KEYSW, K15 KEYSW, K16 KEYSW, K17 KEYSW, K18 KEYSW, K19 KEYSW, K2 KEYSW, K20 KEYSW, K21 KEYSW, K22 KEYSW, K23 KEYSW, K24 KEYSW, K25 KEYSW, K26 KEYSW, K27 KEYSW, K28 KEYSW, K29 KEYSW, K3 KEYSW, K30 KEYSW, K31 KEYSW, K32 KEYSW, K33 KEYSW, K34 KEYSW, K35 KEYSW, K36 KEYSW, K37 KEYSW, K38 KEYSW, K39 KEYSW, K4 KEYSW, K40 KEYSW, K41 KEYSW, K42 KEYSW, K43 KEYSW, K44 KEYSW, K45 KEYSW, K46 KEYSW, K47 KEYSW, K48 KEYSW, K49 KEYSW, K5 KEYSW, K50 KEYSW, K51 KEYSW, K52 KEYSW, K53 KEYSW, K54 KEYSW, K55 KEYSW, K56 KEYSW, K57 KEYSW, K58 KEYSW, K59 KEYSW, K6 KEYSW, K60 KEYSW, K61 KEYSW, K62 KEYSW, K63 KEYSW, K64 KEYSW, K65 KEYSW, K66 KEYSW, K67 KEYSW, K7 KEYSW, K8 KEYSW, K9 KEYSW, U1 ATmega32U4-AU, U2 USBLC6-2SC6, Y1 16MHz

Commit message: v1 ready for review
Parts:
- added C1: 22pF, Capacitor_SMD:C_0805_2012Metric, B.Cu at (106.9, 95.9)
- 6.25 STAB: renamed from >NAME
- C2: value 4.7uF -> 22pF
- D31: value b -> D
- K1, K10, K11, K12, K13, K14, K15, K16, K17, K18, K19, K2, K20, K21, K22, K23, K24, K25, K26, K27, K28, K29, K3, K30, K31, K32, K33, K34, K35, K36, K37, K38, K39, K4, K40, K41, K42, K43, K44, K45, K46, K47, K48, K49, K5, K50, K51, K52, K53, K54, K55, K56, K57, K58, K59, K6, K60, K61, K62, K63, K64, K65, K66, K67, K7, K8, K9: footprint keyboard_parts:Kailh_MX_Socket_LED -> keyboard_parts:Kailh_MX_Socket (3D)
- U2: value USBLC6-2SC6 -> SRV05-4-P-T7
- Y1: value 16MHz -> XTAL; footprint Crystal:Resonator_SMD_muRata_CSTxExxV-3Pin_3.0x1.1mm -> Crystal:Crystal_SMD_3225-4Pin_3.2x2.5mm
- moved C2 103.4 mm to (106.9, 102.4)
- moved R5 18.1 mm to (110.7, 101.7), turned to -90 degrees
- moved C6 6.28 mm to (114.0, 89.6)
- moved C3 2.42 mm to (118.6, 105.8), turned to 180 degrees
- moved R6 1.79 mm to (128.0, 93.0), turned to 90 degrees
- moved C4 1.66 mm to (130.1, 93.0), turned to -90 degrees
- moved Y1 1.65 mm to (106.9, 99.1), turned to 90 degrees
- moved C7 1.22 mm to (127.9, 103.3), turned to -90 degrees
- moved C5 1.06 mm to (123.4, 106.2), turned to 0 degrees
- moved F1 0.94 mm to (35.1, 35.8)
- moved D1 0.80 mm to (20.6, 33.3)
- moved U2 0.58 mm to (34.5, 32.1), turned to 180 degrees
- moved R3 0.25 mm to (39.7, 33.6)
Connections:
- C2 pad 1: VBUS -> GND
- C2 pad 2: GND -> Net-(C2-Pad2)
- C4 pad 1: +5V -> VCC
- C5 pad 1: +5V -> VCC
- C6 pad 1: +5V -> VCC
- C7 pad 1: +5V -> VCC
- J1 pad 5: D- -> DBUS-
- J1 pad 6: D+ -> DBUS+
- J1 pad 7: D- -> DBUS-
- J1 pad 8: D+ -> DBUS+
- Poker_oval_hole pad : (no net) -> GND (x4)
- R3 pad 1: Net-(R3-Pad1) -> DBUS+
- R3 pad 2: Net-(R3-Pad2) -> D+
- R4 pad 1: Net-(R4-Pad1) -> DBUS-
- R4 pad 2: Net-(R4-Pad2) -> D-
- R5 pad 1: +5V -> VCC
- U1 pad 1: Net-(U1-Pad1) -> ROW4
- U1 pad 14: +5V -> VCC
- U1 pad 16: Net-(U1-Pad16) -> Net-(C2-Pad2)
- U1 pad 17: Net-(U1-Pad17) -> Net-(C1-Pad2)
- U1 pad 18: Net-(U1-Pad18) -> COL0
- U1 pad 19: Net-(U1-Pad19) -> COL1
- U1 pad 2: +5V -> VCC
- U1 pad 20: Net-(U1-Pad20) -> COL2
- U1 pad 21: Net-(U1-Pad21) -> COL3
- U1 pad 22: Net-(U1-Pad22) -> ROW3
- U1 pad 24: +5V -> VCC
- U1 pad 25: Net-(U1-Pad25) -> ROW2
- U1 pad 26: Net-(U1-Pad26) -> ROW1
- U1 pad 27: Net-(U1-Pad27) -> ROW0
- U1 pad 28: Net-(U1-Pad28) -> COL4
- U1 pad 29: Net-(U1-Pad29) -> COL5
- U1 pad 3: Net-(R4-Pad2) -> D-
- U1 pad 30: Net-(U1-Pad30) -> COL6
- U1 pad 31: Net-(U1-Pad31) -> COL7
- U1 pad 32: Net-(U1-Pad32) -> COL8
- U1 pad 34: +5V -> VCC
- U1 pad 36: Net-(U1-Pad36) -> COL14
- U1 pad 37: Net-(U1-Pad37) -> COL13
- U1 pad 38: Net-(U1-Pad38) -> COL12
- U1 pad 39: Net-(U1-Pad39) -> COL11
- U1 pad 4: Net-(R3-Pad2) -> D+
- U1 pad 40: Net-(U1-Pad40) -> COL10
- U1 pad 41: Net-(U1-Pad41) -> COL9
- U1 pad 44: +5V -> VCC
- U1 pad 7: +5V -> VCC
- U2 pad 1: D- -> DBUS+
- U2 pad 3: D+ -> DBUS+
- U2 pad 4: Net-(R3-Pad1) -> DBUS-
- U2 pad 6: Net-(R4-Pad1) -> DBUS-
- Y1 pad 1: Net-(U1-Pad17) -> Net-(C2-Pad2)
- Y1 pad 2: Net-(U1-Pad16) -> GND
- Y1 pad 3: GND -> Net-(C1-Pad2)
Routing:
- net COL13: track 0.00 -> 263.9 mm, vias 0 -> 4
- net COL12: track 0.00 -> 257.6 mm, vias 0 -> 4
- net COL11: track 0.00 -> 240.2 mm, vias 0 -> 5
- net COL10: track 0.00 -> 231.4 mm, vias 0 -> 5
- net VCC: track 35.9 -> 256.7 mm, vias 0 -> 6
- net COL14: track 80.4 -> 291.1 mm, vias 0 -> 5
- net COL9: track 0.00 -> 200.0 mm, vias 0 -> 5
- net COL8: track 0.00 -> 167.5 mm, vias 0 -> 5
- net D+: track 11.0 -> 170.5 mm, vias 0 -> 2
- net D-: track 16.3 -> 171.7 mm, vias 0 -> 2
- net COL7: track 0.00 -> 152.8 mm, vias 0 -> 5
- net COL5: track 0.00 -> 138.1 mm, vias 0 -> 6
- net COL6: track 0.00 -> 135.2 mm, vias 0 -> 5
- net COL2: track 0.00 -> 131.7 mm, vias 0 -> 6
- net COL1: track 33.3 -> 163.4 mm, vias 2 -> 6
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- added copper zone on B.Cu, net GND

Commit message: v1.0a update
Parts:
- added C10: 0.1uF, Capacitor_SMD:C_0805_2012Metric, B.Cu at (91.3, 106.4)
- added C11: 0.1uF, Capacitor_SMD:C_0805_2012Metric, B.Cu at (151.6, 106.4)
- added C12: 0.1uF, Capacitor_SMD:C_0805_2012Metric, B.Cu at (173.0, 106.5)
- added C13: 0.1uF, Capacitor_SMD:C_0805_2012Metric, B.Cu at (184.9, 106.4)
- added C14: 0.1uF, Capacitor_SMD:C_0805_2012Metric, B.Cu at (254.8, 106.4)
- added C15: 0.1uF, Capacitor_SMD:C_0805_2012Metric, B.Cu at (280.1, 106.4)
- added C8: 4.7nF, Capacitor_SMD:C_0805_2012Metric, B.Cu at (42.0, 20.2)
- added C9: 0.1uF, Capacitor_SMD:C_0805_2012Metric, B.Cu at (65.9, 106.5)
- added J2: AVR-ISP-6, random-keyboard-parts:Reset_Pretty-Mask, B.Cu at (91.1, 98.7)
- added R7: 1M, Resistor_SMD:R_0805_2012Metric, B.Cu at (27.8, 20.2)
- added RGB1: SK6812, LED_SMD:LED_SK6812_PLCC4_5.0x5.0mm_P3.2mm, B.Cu at (61.1, 106.4)
- added RGB2: SK6812, LED_SMD:LED_SK6812_PLCC4_5.0x5.0mm_P3.2mm, B.Cu at (86.5, 106.4)
- added RGB3: SK6812, LED_SMD:LED_SK6812_PLCC4_5.0x5.0mm_P3.2mm, B.Cu at (146.8, 106.4)
- added RGB4: SK6812, LED_SMD:LED_SK6812_PLCC4_5.0x5.0mm_P3.2mm, B.Cu at (168.3, 106.4)
- added RGB5: SK6812, LED_SMD:LED_SK6812_PLCC4_5.0x5.0mm_P3.2mm, B.Cu at (189.7, 106.4)
- added RGB6: SK6812, LED_SMD:LED_SK6812_PLCC4_5.0x5.0mm_P3.2mm, B.Cu at (250.0, 106.4)
- added RGB7: SK6812, LED_SMD:LED_SK6812_PLCC4_5.0x5.0mm_P3.2mm, B.Cu at (275.4, 106.4)
- added athene logo: LOGO, Graphics:athene, B.Cu at (175.0, 96.8)
- added kl logo: LOGO, Graphics:kl, F.Cu at (173.0, 101.6)
- K29, K37, K60, K66: footprint keyboard_parts:Kailh_MX_Socket (3D) -> keyboard_parts:Kailh_MX_Socket (3D) 1_Circle
- ST_ENTER: renamed from >NAME; value >VALUE -> Stabilizer
- ST_SPACE: renamed from 6.25 STAB; value >VALUE -> Stabilizer
- moved S1 106.3 mm to (55.4, 81.0), turned to 90 degrees
- moved C7 19.9 mm to (113.5, 89.5), turned to 180 degrees
- moved C5 17.7 mm to (127.3, 101.2), turned to 90 degrees
- moved C4 14.4 mm to (123.7, 105.9), turned to 0 degrees
- moved C6 14.3 mm to (127.4, 92.5), turned to -90 degrees
- moved D37 9.82 mm to (147.6, 67.5), turned to 90 degrees
- moved D29 9.68 mm to (281.0, 48.3), turned to 90 degrees
- moved D59 8.73 mm to (20.2, 94.5), turned to -90 degrees
- moved D62 7.49 mm to (138.1, 96.0), turned to 0 degrees
- moved D64 7.24 mm to (240.5, 96.0), turned to 0 degrees
- moved D67 7.24 mm to (302.4, 96.0), turned to 0 degrees
- moved D61 7.24 mm to (66.7, 96.0), turned to 0 degrees
- moved D63 7.24 mm to (211.9, 96.0), turned to 0 degrees
- moved D65 7.24 mm to (264.3, 96.0), turned to 0 degrees
- moved R6 3.55 mm to (126.6, 89.7), turned to 180 degrees
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- renumbered C6 to C5, C5 to C6, ST72 to ST_BKSP, ST72 to ST_LSHIFT
Connections:
- J1 pad 13: GND -> Net-(C8-Pad1)
- U1 pad 10: Net-(U1-Pad10) -> MOSI
- U1 pad 11: Net-(U1-Pad11) -> MISO
- U1 pad 12: Net-(U1-Pad12) -> RGB
- U1 pad 25: ROW2 -> ROW0
- U1 pad 27: ROW0 -> ROW2
- U1 pad 36: COL14 -> COL9
- U1 pad 37: COL13 -> COL10
- U1 pad 38: COL12 -> COL11
- U1 pad 39: COL11 -> COL12
- U1 pad 40: COL10 -> COL13
- U1 pad 41: COL9 -> COL14
- U1 pad 9: Net-(U1-Pad9) -> SCLK
Routing:
- net VCC: track 256.7 -> 439.6 mm, vias 6 -> 12
- net Net-(RGB2-Pad4): track 0.00 -> 69.2 mm, vias 0 -> 2
- net Net-(RGB5-Pad4): track 0.00 -> 66.7 mm, vias 0 -> 2
- net RGB: track 0.00 -> 53.2 mm, vias 0 -> 3
- net GND: track 118.6 -> 166.1 mm, vias 2 -> 6
- net MOSI: track 0.00 -> 35.9 mm, vias 0 -> 1
- net SCLK: track 0.00 -> 33.5 mm, vias 0 -> 1
- net Net-(RGB6-Pad4): track 0.00 -> 32.4 mm, vias 0 -> 2
- net MISO: track 0.00 -> 32.0 mm, vias 0 -> 1
- net Net-(RGB1-Pad4): track 0.00 -> 31.6 mm, vias 0 -> 2
- net D-: track 171.7 -> 141.6 mm
- net D+: track 170.5 -> 140.7 mm
- net Net-(RGB4-Pad4): track 0.00 -> 29.2 mm, vias 0 -> 2
- net Net-(RGB3-Pad4): track 0.00 -> 27.6 mm, vias 0 -> 2
- net Net-(C8-Pad1): track 0.00 -> 22.8 mm
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Other:
- board text added: "rev. 1.0a | designed by kl"

Commit message: v1.0a update
Parts:
- K1, K10, K11, K12, K13, K14, K15, K16, K17, K18, K19, K2, K20, K21, K22, K23, K24, K25, K26, K27, K28, K3, K30, K31, K32, K33, K34, K35, K36, K38, K39, K4, K40, K41, K42, K43, K44, K45, K46, K47, K48, K49, K5, K50, K51, K52, K53, K54, K55, K56, K57, K58, K59, K6, K61, K62, K63, K64, K65, K67, K7, K8, K9: footprint keyboard_parts:Kailh_MX_Socket (3D) -> Project Library:Kailh_MX_Socket (3D)
- K29, K37, K60, K66: footprint keyboard_parts:Kailh_MX_Socket (3D) 1_Circle -> Project Library:Kailh_MX_Socket (3D) 1_Circle
